File: TRNG.sch (EAGLE design)
At the start: 9 parts

Commit message: update
Other:
- note added: "True Random Number Generator (TRNG) Copyright (C) 2020 Manny Peterson <me@mannypeterson.com>"
- note removed: "spicy-bits.org True Random Number Generator (TRNG) Copyright (C) 2020 Manny Peterson <me@mannypeterson.com>"
Changed lines of the file:
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@@
 <sheet>
 <plain>
-<text x="96.52" y="86.36" size="1.778" layer="91">spicy-bits.org True Random Number Generator (TRNG)
+<text x="127" y="83.82" size="1.778" layer="91" align="center">True Random Number Generator (TRNG)
 Copyright (C) 2020 Manny Peterson &lt;me@mannypeterson.com&gt;</text>
 </plain>
